File: AMS1117.sch (KiCad schematic (older format))
At the start: 11 parts

Commit message: update,
Parts:
- removed JP?: IN_EN, symbol Device:Jumper_NO_Small
- removed JP?: OUT_EN, symbol Device:Jumper_NO_Small
- added JP?: IN_EN, Jumper:SolderJumper-2_P1.3mm_Open_RoundedPad1.0x1.5mm, symbol my_solder_jumper:SolderJumper_2_Open_round
- added JP?: OUT_EN, Jumper:SolderJumper-2_P1.3mm_Open_RoundedPad1.0x1.5mm, symbol my_solder_jumper:SolderJumper_2_Open_round
Connections:
- net +3V3: now also JP?.1 (A)
- net +5V: now also JP?.1 (A)
- net at C?.1, C?.1, U?.2 (VO): now also JP?.2 (B)
- net at C?.1, U?.3 (VI): now also JP?.2 (B)
Changed lines of the file:
@@
 L power:+3V3 #PWR?
 U 1 1 5C0C0902
-P 3700 1500
-F 0 "#PWR?" H 3700 1350 50  0001 C CNN
-F 1 "+3V3" H 3750 1700 50  0000 C CNN
-F 2 "" H 3700 1500 50  0001 C CNN
-F 3 "" H 3700 1500 50  0001 C CNN
-	1    3700 1500
+P 3700 1400
+F 0 "#PWR?" H 3700 1250 50  0001 C CNN
+F 1 "+3V3" H 3750 1600 50  0000 C CNN
+F 2 "" H 3700 1400 50  0001 C CNN
+F 3 "" H 3700 1400 50  0001 C CNN
+	1    3700 1400
 	1    0    0    -1
 $EndComp
@@
 	0    -1   -1   0
 $EndComp
-$Comp
-L Device:Jumper_NO_Small JP?
-U 1 1 5C148323
-P 2250 1700
-F 0 "JP?" V 2200 1750 50  0000 L CNN
-F 1 "IN_EN" V 2250 1750 50  0000 L CNN
-F 2 "" H 2250 1700 50  0001 C CNN
-F 3 "~" H 2250 1700 50  0001 C CNN
-	1    2250 1700
-	0    1    1    0
-$EndComp
-Wire Wire Line
-	2250 1550 2250 1600
+Wire Wire Line
+	2250 1400 2250 1500
 Wire Wire Line
 	2250 1800 2250 1950
-$Comp
-L Device:Jumper_NO_Small JP?
-U 1 1 5C148F3B
-P 3700 1700
-F 0 "JP?" V 3650 1750 50  0000 L CNN
-F 1 "OUT_EN" V 3700 1750 50  0000 L CNN
-F 2 "" H 3700 1700 50  0001 C CNN
-F 3 "~" H 3700 1700 50  0001 C CNN
-	1    3700 1700
-	0    1    1    0
-$EndComp
 Wire Wire Line
 	3700 1800 3700 1950
@@
 L power:+5V #PWR?
 U 1 1 5C153651
-P 2250 1550
-F 0 "#PWR?" H 2250 1400 50  0001 C CNN
-F 1 "+5V" H 2300 1750 50  0000 C CNN
-F 2 "" H 2250 1550 50  0001 C CNN
-F 3 "" H 2250 1550 50  0001 C CNN
-	1    2250 1550
-	1    0    0    -1
-$EndComp
-Wire Wire Line
-	3700 1500 3700 1600
+P 2250 1400
+F 0 "#PWR?" H 2250 1250 50  0001 C CNN
+F 1 "+5V" H 2300 1600 50  0000 C CNN
+F 2 "" H 2250 1400 50  0001 C CNN
+F 3 "" H 2250 1400 50  0001 C CNN
+	1    2250 1400
+	1    0    0    -1
+$EndComp
+Wire Wire Line
+	3700 1400 3700 1500
 $Comp
 L power:+3V3 #PWR?
@@
 Wire Wire Line
 	2950 3550 2950 3750
+$Comp
+L my_solder_jumper:SolderJumper_2_Open_round JP?
+U 1 1 5D072C46
+P 2250 1650
+F 0 "JP?" V 2204 1718 50  0000 L CNN
+F 1 "IN_EN" V 2295 1718 50  0000 L CNN
+F 2 "Jumper:SolderJumper-2_P1.3mm_Open_RoundedPad1.0x1.5mm" H 2250 1650 50  0001 C CNN
+F 3 "~" H 2250 1650 50  0001 C CNN
+	1    2250 1650
+	0    1    1    0
+$EndComp
+$Comp
+L my_solder_jumper:SolderJumper_2_Open_round JP?
+U 1 1 5D077B21
+P 3700 1650
+F 0 "JP?" V 3654 1718 50  0000 L CNN
+F 1 "OUT_EN" V 3745 1718 50  0000 L CNN
+F 2 "Jumper:SolderJumper-2_P1.3mm_Open_RoundedPad1.0x1.5mm" H 3700 1650 50  0001 C CNN
+F 3 "~" H 3700 1650 50  0001 C CNN
+	1    3700 1650
+	0    1    1    0
+$EndComp
 $EndSCHEMATC

Commit message: updaste,
Parts:
- D?: value LED_GREEN,0603 -> 3V3_HEALTHY
Changed lines of the file:
@@
 P 2250 3550
 F 0 "D?" V 2300 3450 50  0000 R CNN
-F 1 "LED_GREEN,0603" V 2250 3450 50  0000 R CNN
+F 1 "3V3_HEALTHY" V 2250 3450 50  0000 R CNN
 F 2 "LED_SMD:LED_0603_1608Metric_Pad1.05x0.95mm_HandSolder" V 2250 3550 50  0001 C CNN
 F 3 "" V 2250 3550 50  0001 C CNN
